File: SchematicsAndPCBs/Full System/Full Battery System.sch (KiCad schematic (older format))
At the start: 19 parts, among them K1 DPST Relay, SW1 ChargeSwitch, SW2 RTDSwitch (latch), U1 OrionCurrentSens, U2 OrionBMS2, U3 OrionThermExp, U4 OrionThermExp

Commit message: Parts library System Updates
>Added Kicad libraries folder to SchematicsandPCBs
>Added NER parts library to KiCAD folder
>Moved all custom parts to new NER library
>Deleted old random libraries
Parts:
- removed U?: TSM2500, symbol Full-Battery-System-rescue:TSM2500-FSAE_Components
- added U?: TSM2500, symbol NER:TSM2500
Changed lines of the file:
@@
 $EndDescr
-$Comp
-L Full-Battery-System-rescue:TSM2500-FSAE_Components U?
-U 1 1 5DC5A085
-P 3100 1200
-F 0 "U?" H 3100 1200 50  0001 C CNN
-F 1 "TSM2500" H 3125 1223 50  0000 C CNN
-F 2 "" H 3100 1200 50  0001 C CNN
-F 3 "" H 3100 1200 50  0001 C CNN
-	1    3100 1200
-	1    0    0    -1
-$EndComp
 $Comp
 L Device:Battery BT2
@@
 Wire Wire Line
 	1600 7450 2350 7450
+$Comp
+L NER:TSM2500 U?
+U 1 1 5F581E55
+P 3100 1200
+F 0 "U?" H 3100 1200 50  0001 C CNN
+F 1 "TSM2500" H 3125 1223 50  0000 C CNN
+F 2 "" H 3100 1200 50  0001 C CNN
+F 3 "" H 3100 1200 50  0001 C CNN
+	1    3100 1200
+	1    0    0    -1
+$EndComp
 $EndSCHEMATC
