File: SchematicsAndPCBs/Master System Schematic/Charger.sch (KiCad schematic (older format))
At the start: 5 parts

Commit message: Updating Library References
Shifting references in the Master Schematic project to use the new NER library
Parts:
- U?: symbol Charger-rescue:TSM2500-FSAE_Components -> NER:TSM2500
Changed lines of the file:
@@
 EESchema Schematic File Version 4
+LIBS:Master System Schematic-cache
 EELAYER 30 0
 EELAYER END
@@
 $EndComp
 $Comp
-L Charger-rescue:TSM2500-FSAE_Components U?
+L NER:TSM2500 U?
 U 1 1 61EEF410
 P 5550 4350
