File: SchematicsAndPCBs/Master System Schematic/Shutdown_LatchingCircuits.sch (KiCad schematic (older format))
At the start: 6 parts, among them K1 3PoleSwitchingRelay, K2 3PoleSwitchingRelay, SW5 IMD_LatchReset, SW6 BMS_LatchReset

Commit message: Updating Library References
Shifting references in the Master Schematic project to use the new NER library
Parts:
- K1, K2: symbol Shutdown-rescue:3PoleSwitchingRelay-FSAE_Components -> NER:3PoleSwitchingRelay
Changed lines of the file:
@@
 EESchema Schematic File Version 4
+LIBS:Master System Schematic-cache
 EELAYER 30 0
 EELAYER END
@@
 $EndComp
 $Comp
-L Shutdown-rescue:3PoleSwitchingRelay-FSAE_Components K2
+L NER:3PoleSwitchingRelay K2
 U 1 1 5DE0D324
 P 7350 2500
+AR Path="/5DE0D324" Ref="K2"  Part="1"
+AR Path="/5F45AFB3/5DE0D324" Ref="K2"  Part="1"
 F 0 "K2" H 7350 2615 50  0000 C CNN
 F 1 "3PoleSwitchingRelay" H 7350 2524 50  0000 C CNN
@@
 $EndComp
 $Comp
-L Shutdown-rescue:3PoleSwitchingRelay-FSAE_Components K1
+L NER:3PoleSwitchingRelay K1
 U 1 1 5DDDA065
 P 4150 2400
+AR Path="/5DDDA065" Ref="K1"  Part="1"
+AR Path="/5F45AFB3/5DDDA065" Ref="K1"  Part="1"
 F 0 "K1" H 4150 2515 50  0000 C CNN
 F 1 "3PoleSwitchingRelay" H 4150 2424 50  0000 C CNN
