File: Schematics/Master System Schematic/Driver IO Enclosure.sch (KiCad schematic (older format))
At the start: 1 part

Commit message: Added GLV Fusebox component
Made fusebox component, and added to master schematic
Parts:
- removed SW?: Cockpit Shutdown (BRB), symbol Switch:SW_Push_Open
Changed lines of the file:
@@
 EESchema Schematic File Version 4
-LIBS:Master System Schematic-cache
 EELAYER 30 0
 EELAYER END
@@
 Comment4 ""
 $EndDescr
-$Comp
-L Switch:SW_Push_Open SW?
-U 1 1 5F67335D
-P 5400 3300
-AR Path="/5F45AFB3/5F67335D" Ref="SW?"  Part="1"
-AR Path="/5F67335D" Ref="SW?"  Part="1"
-AR Path="/5F670E17/5F67335D" Ref="SW?"  Part="1"
-AR Path="/5F647A32/5F67335D" Ref="SW?"  Part="1"
-F 0 "SW?" V 5446 3247 50  0000 R CNN
-F 1 "Cockpit Shutdown (BRB)" V 5355 3247 50  0000 R CNN
-F 2 "" H 5400 3500 50  0001 C CNN
-F 3 "~" H 5400 3500 50  0001 C CNN
-	1    5400 3300
-	0    1    1    0
-$EndComp
 $EndSCHEMATC
