File: Schematics/Master System Schematic/Master System Schematic.sch (KiCad schematic (older format))
At the start: 33 parts, among them J1 GND, J2 TS+, J3 TS-, SW1 GLVMS, SW2 SideMounted (BRB), SW3 SideMounted (BRB)

Commit message: Connectors and Start of Numbering
Created new generic connectors and applied numbering tool to whole project
Parts:
- gave numbers to parts that had none: 25
Connections:
- new net: U3.6, U6.23 (CANB_H), U6.8 (Reverse_Enable_Switch)
- new net: U6.~ (TS-), U7.~ (AC3) (x2)
- now unconnected: U6.23 (CANB_H), U6.8 (Reverse_Enable_Switch)
Changed lines of the file:
@@
 EESchema Schematic File Version 4
+LIBS:Master System Schematic-cache
 EELAYER 30 0
 EELAYER END
@@
 P 2300 3200
 AR Path="/5F45AFB3/5F633AC3" Ref="SW?"  Part="1"
-AR Path="/5F633AC3" Ref="SW?"  Part="1"
-F 0 "SW?" V 2300 2650 50  0000 C CNN
+AR Path="/5F633AC3" Ref="SW4"  Part="1"
+F 0 "SW4" V 2300 2650 50  0000 C CNN
 F 1 "Brake Over-Travel Switch" V 2200 2600 50  0000 C CNN
 F 2 "" H 2300 3200 50  0001 C CNN
@@
 P 5950 3350
 AR Path="/5F45AFB3/5F67997D" Ref="SW?"  Part="1"
-AR Path="/5F67997D" Ref="SW?"  Part="1"
-F 0 "SW?" V 6000 3600 50  0000 R CNN
+AR Path="/5F67997D" Ref="SW6"  Part="1"
+F 0 "SW6" V 6000 3600 50  0000 R CNN
 F 1 "Cockpit Shutdown (BRB)" V 5900 4350 50  0000 R CNN
 F 2 "" H 5950 3550 50  0001 C CNN
@@
 P 5950 4600
 AR Path="/5F45AFB3/5F67998A" Ref="SW?"  Part="1"
-AR Path="/5F67998A" Ref="SW?"  Part="1"
-F 0 "SW?" V 5904 4698 50  0000 L CNN
+AR Path="/5F67998A" Ref="SW7"  Part="1"
+F 0 "SW7" V 5904 4698 50  0000 L CNN
 F 1 "TSMS" V 5995 4698 50  0000 L CNN
 F 2 "" H 5950 4600 50  0001 C CNN
@@
 P 6200 2350
 AR Path="/5F45AFB3/5F67996F" Ref="D?"  Part="1"
-AR Path="/5F67996F" Ref="D?"  Part="1"
-F 0 "D?" H 6193 2095 50  0000 C CNN
+AR Path="/5F67996F" Ref="D4"  Part="1"
+F 0 "D4" H 6193 2095 50  0000 C CNN
 F 1 "SSOK1" H 6193 2186 50  0000 C CNN
 F 2 "" H 6200 2350 50  0001 C CNN
@@
 P 6200 1950
 AR Path="/5F45AFB3/5F679969" Ref="D?"  Part="1"
-AR Path="/5F679969" Ref="D?"  Part="1"
-F 0 "D?" H 6193 1695 50  0000 C CNN
+AR Path="/5F679969" Ref="D3"  Part="1"
+F 0 "D3" H 6193 1695 50  0000 C CNN
 F 1 "SSOK2" H 6193 1786 50  0000 C CNN
 F 2 "" H 6200 1950 50  0001 C CNN
@@
 $EndComp
 $Comp
-L NER:Bender_Isometer_IR155-3204 U?
+L NER:Bender_Isometer_IR155-3204 U4
 U 1 1 5F94A015
 P 7600 3800
-F 0 "U?" H 7600 3915 50  0000 C CNN
+F 0 "U4" H 7600 3915 50  0000 C CNN
 F 1 "Bender_Isometer_IR155-3204" H 7600 3824 50  0000 C CNN
 F 2 "" H 7600 3800 50  0001 C CNN
@@
 	6550 2150 6550 1950
 $Comp
-L Device:R R?
+L Device:R R5
 U 1 1 5F4E06AE
 P 7600 3500
-F 0 "R?" V 7807 3500 50  0000 C CNN
+F 0 "R5" V 7807 3500 50  0000 C CNN
 F 1 "2.2k" V 7716 3500 50  0000 C CNN
 F 2 "" V 7530 3500 50  0001 C CNN
@@
 CHASSIS_GND
 $Comp
-L NER:OrionCurrentSens U?
+L NER:OrionCurrentSens U5
 U 1 1 6111F589
 P 9350 8050
-F 0 "U?" H 9350 8050 50  0000 C CNN
+F 0 "U5" H 9350 8050 50  0000 C CNN
 F 1 "OrionCurrentSens" H 9350 8100 50  0000 C CNN
 F 2 "" H 9350 8050 50  0001 C CNN
@@
 CHASSIS_GND
 $Comp
-L NER:FuseBox_PSZACCEPS052H U?
+L NER:FuseBox_PSZACCEPS052H U3
 U 1 1 5F6D724E
 P 1250 3250
-F 0 "U?" H 1250 3415 50  0000 C CNN
+F 0 "U3" H 1250 3415 50  0000 C CNN
 F 1 "FuseBox_PSZACCEPS052H" H 1250 3324 50  0000 C CNN
 F 2 "" H 1250 3400 50  0001 C CNN
@@
 	1250 4150 1250 4500
 $Comp
-L Device:LED D?
+L Device:LED D1
 U 1 1 5F90AC4F
 P 2550 1500
-F 0 "D?" H 2543 1716 50  0000 C CNN
+F 0 "D1" H 2543 1716 50  0000 C CNN
 F 1 "IMD Fault Indicator" H 2543 1625 50  0000 C CNN
 F 2 "" H 2550 1500 50  0001 C CNN
@@
 $EndComp
 $Comp
-L Device:LED D?
+L Device:LED D2
 U 1 1 5F90FD2E
 P 2550 1900
-F 0 "D?" H 2550 1800 50  0000 C CNN
+F 0 "D2" H 2550 1800 50  0000 C CNN
 F 1 "BMS Fault Indicator" H 2550 1700 50  0000 C CNN
 F 2 "" H 2550 1900 50  0001 C CNN
@@
 Connection ~ 8650 7900
 $Comp
-L Device:LED D?
+L Device:LED D5
 U 1 1 5FA58D8C
 P 6300 5500
-F 0 "D?" H 6250 5400 50  0000 L CNN
+F 0 "D5" H 6250 5400 50  0000 L CNN
 F 1 "TSAL" H 6250 5300 50  0000 L CNN
 F 2 "" H 6300 5500 50  0001 C CNN
@@
 	15350 1000 15350 7900
 $Comp
-L NER:RinehartPM100DX_MotorController U?
+L NER:RinehartPM100DX_MotorController U6
 U 1 1 5F97D518
 P 14300 8350
-F 0 "U?" H 14300 8515 50  0000 C CNN
+F 0 "U6" H 14300 8515 50  0000 C CNN
 F 1 "RinehartPM100DX_MotorController" H 14300 8424 50  0000 C CNN
 F 2 "" H 14300 8350 50  0001 C CNN
@@
 $EndComp
 $Comp
-L Device:R_POT RV?
+L Device:R_POT RV4
 U 1 1 6233DFFE
 P 13050 7750
-F 0 "RV?" H 12800 7850 50  0000 C CNN
+F 0 "RV4" H 12800 7850 50  0000 C CNN
 F 1 "ACCEL_POT" H 12800 7750 50  0000 C CNN
 F 2 "" H 13050 7750 50  0001 C CNN
@@
 $EndComp
 $Comp
-L Device:R_POT RV?
+L Device:R_POT RV3
 U 1 1 6233F5CA
 P 13050 7350
-F 0 "RV?" H 12800 7450 50  0000 C CNN
+F 0 "RV3" H 12800 7450 50  0000 C CNN
 F 1 "BRAKE_POT" H 12800 7350 50  0000 C CNN
 F 2 "" H 13050 7350 50  0001 C CNN
@@
 $EndComp
 $Comp
-L Switch:SW_SPST SW?
+L Switch:SW_SPST SW11
 U 1 1 62347AF0
 P 13050 6200
-F 0 "SW?" H 13050 5975 50  0000 C CNN
+F 0 "SW11" H 13050 5975 50  0000 C CNN
 F 1 "BRAKE_SWITCH" H 13050 6066 50  0000 C CNN
 F 2 "" H 13050 6200 50  0001 C CNN
@@
 	15750 8250 15750 8300
 $Comp
-L NER:Emrax228HV_Motor U?
+L NER:Emrax228HV_Motor U7
 U 1 1 5F972C2B
 P 16100 7800
-F 0 "U?" H 16050 7950 50  0000 L CNN
+F 0 "U7" H 16050 7950 50  0000 L CNN
 F 1 "Emrax228HV_Motor" H 15750 7850 50  0000 L CNN
 F 2 "" H 16100 7800 50  0001 C CNN
@@
 	6100 8050 6100 8450
 $Comp
-L Switch:SW_DPST SW?
+L Switch:SW_DPST SW5
 U 1 1 5F864268
 P 4950 8250
-F 0 "SW?" H 4950 8050 50  0000 C CNN
+F 0 "SW5" H 4950 8050 50  0000 C CNN
 F 1 "Latching Circuit Reset [Momentary Button NO]" H 4500 7900 50  0000 C CNN
 F 2 "" H 4950 8250 50  0001 C CNN
@@
 	1850 3950 6900 3950
 $Comp
-L Switch:SW_SPST_Temperature SW?
+L Switch:SW_SPST_Temperature SW12
 U 1 1 5F6E407C
 P 14850 3700
-F 0 "SW?" H 14850 4015 50  0000 C CNN
+F 0 "SW12" H 14850 4015 50  0000 C CNN
 F 1 "SW_SPST_Pressure" H 14850 3924 50  0000 C CNN
 F 2 "" H 14850 3700 50  0001 C CNN
@@
 $EndComp
 $Comp
-L Switch:SW_SPST_Temperature SW?
+L Switch:SW_SPST_Temperature SW13
 U 1 1 5F6E49B5
 P 14850 4200
-F 0 "SW?" H 14850 4515 50  0000 C CNN
+F 0 "SW13" H 14850 4515 50  0000 C CNN
 F 1 "SW_SPST_Pressure" H 14850 4424 50  0000 C CNN
 F 2 "" H 14850 4200 50  0001 C CNN
@@
 $EndSheet
 $Comp
-L Device:R_POT RV?
+L Device:R_POT RV2
 U 1 1 5F71DF92
 P 12450 4150
-F 0 "RV?" H 12381 4196 50  0000 R CNN
+F 0 "RV2" H 12381 4196 50  0000 R CNN
 F 1 "R_POT" H 12381 4105 50  0000 R CNN
 F 2 "" H 12450 4150 50  0001 C CNN
@@
 $EndComp
 $Comp
-L Device:R_POT RV?
+L Device:R_POT RV1
 U 1 1 5F71E67B
 P 12450 3650
-F 0 "RV?" H 12381 3696 50  0000 R CNN
+F 0 "RV1" H 12381 3696 50  0000 R CNN
 F 1 "R_POT" H 12381 3605 50  0000 R CNN
 F 2 "" H 12450 3650 50  0001 C CNN
@@
 P 6250 6400
 AR Path="/5F45B05E/60DA2E32" Ref="SW?"  Part="1"
-AR Path="/60DA2E32" Ref="SW?"  Part="1"
-F 0 "SW?" H 6250 6550 50  0000 C CNN
+AR Path="/60DA2E32" Ref="SW9"  Part="1"
+F 0 "SW9" H 6250 6550 50  0000 C CNN
 F 1 "HVD" H 6250 6650 50  0000 C CNN
 F 2 "" H 6250 6400 50  0001 C CNN
@@
 P 6250 6000
 AR Path="/5F45B05E/60DA2E38" Ref="SW?"  Part="1"
-AR Path="/60DA2E38" Ref="SW?"  Part="1"
-F 0 "SW?" H 6250 6235 50  0000 C CNN
+AR Path="/60DA2E38" Ref="SW8"  Part="1"
+F 0 "SW8" H 6250 6235 50  0000 C CNN
 F 1 "SMD" H 6250 6144 50  0000 C CNN
 F 2 "" H 6250 6000 50  0001 C CNN
@@
 P 6250 6800
 AR Path="/5F45B05E/60DA2E3E" Ref="SW?"  Part="1"
-AR Path="/60DA2E3E" Ref="SW?"  Part="1"
-F 0 "SW?" H 6250 6950 50  0000 C CNN
+AR Path="/60DA2E3E" Ref="SW10"  Part="1"
+F 0 "SW10" H 6250 6950 50  0000 C CNN
 F 1 "SMD" H 6250 7050 50  0000 C CNN
 F 2 "" H 6250 6800 50  0001 C CNN
