File: Schematics/Master System Schematic/Charger.sch (KiCad schematic (older format))
At the start: 5 parts, among them J9 WallSocket, K11 Safety Relay, U8 TSM2500

Commit message: Revert "Driver IO Update"
This reverts commit 719adb322f5430e89ce6e16a8f4347f22c153558.
Parts:
- U8: symbol Master-System-Schematic-rescue:TSM2500-NER -> NER:TSM2500
Changed lines of the file:
@@
 EESchema Schematic File Version 4
+LIBS:Master System Schematic-cache
 EELAYER 30 0
 EELAYER END
@@
 $EndComp
 $Comp
-L Master-System-Schematic-rescue:TSM2500-NER U?
+L NER:TSM2500 U?
 U 1 1 61EEF410
 P 5550 4350

Commit message: Driver IO Update
Added Arduino to enclosure
Parts:
- U8: symbol NER:TSM2500 -> Master-System-Schematic-rescue:TSM2500-NER
Changed lines of the file:
@@
 EESchema Schematic File Version 4
-LIBS:Master System Schematic-cache
 EELAYER 30 0
 EELAYER END
@@
 $EndComp
 $Comp
-L NER:TSM2500 U?
+L Master-System-Schematic-rescue:TSM2500-NER U?
 U 1 1 61EEF410
 P 5550 4350
