File: Schematics/Master System Schematic/PedalBox.sch (KiCad schematic (older format))
At the start: 4 parts, among them U9 CAN_Bus_Module

Commit message: Driver IO Update
Added Arduino to enclosure
Parts:
- A1: symbol NER:Arduino_UNO_rev3 -> Master-System-Schematic-rescue:Arduino_UNO_rev3-NER
- U9: symbol NER:CAN_Bus_Module -> Master-System-Schematic-rescue:CAN_Bus_Module-NER
Connections:
- new net: A1.~ (~~D9), U9.~ (Serial_Clock) (x5)
Changed lines of the file:
@@
 EESchema Schematic File Version 4
-LIBS:Master System Schematic-cache
 EELAYER 30 0
 EELAYER END
@@
 	3600 3050 4350 3050
 $Comp
-L NER:Arduino_UNO_rev3 A1
+L Master-System-Schematic-rescue:Arduino_UNO_rev3-NER A1
 U 1 1 5F6833F8
 P 4950 2900
@@
 NoConn ~ 4350 4150
 $Comp
-L NER:CAN_Bus_Module U9
+L Master-System-Schematic-rescue:CAN_Bus_Module-NER U9
 U 1 1 5F6D982E
 P 7600 3200

Commit message: Revert "Driver IO Update"
This reverts commit 719adb322f5430e89ce6e16a8f4347f22c153558.
Parts:
- A1: symbol Master-System-Schematic-rescue:Arduino_UNO_rev3-NER -> NER:Arduino_UNO_rev3
- U9: symbol Master-System-Schematic-rescue:CAN_Bus_Module-NER -> NER:CAN_Bus_Module
Connections:
- new net: A1.~ (~~D9), U9.~ (Serial_Clock) (x5)
Changed lines of the file:
@@
 EESchema Schematic File Version 4
+LIBS:Master System Schematic-cache
 EELAYER 30 0
 EELAYER END
@@
 	3600 3050 4350 3050
 $Comp
-L Master-System-Schematic-rescue:Arduino_UNO_rev3-NER A1
+L NER:Arduino_UNO_rev3 A1
 U 1 1 5F6833F8
 P 4950 2900
@@
 NoConn ~ 4350 4150
 $Comp
-L Master-System-Schematic-rescue:CAN_Bus_Module-NER U9
+L NER:CAN_Bus_Module U9
 U 1 1 5F6D982E
 P 7600 3200
