File: Schematics/Master System Schematic/PedalBox.sch (KiCad schematic (older format))
At the start: 4 parts, among them U9 CAN_Bus_Module

Commit message: Cooling Pump, TSMP container Updates
>Added Cooling pump relay
>Added Cooling pump
>Added +12V plug to TSMP container
Connections:
- new net: A1.~ (~~D9), U9.~ (Serial_Clock) (x5)
Changed lines of the file:
@@
 EESchema Schematic File Version 4
-LIBS:Master System Schematic-cache
 EELAYER 30 0
 EELAYER END

Commit message: Started Voltage tap pcbs
Connections:
- new net: A1.~ (~~D9), U9.~ (Serial_Clock) (x5)
Changed lines of the file:
@@
 $Descr A 11000 8500
 encoding utf-8
-Sheet 12 13
+Sheet 12 17
 Title "Pedal Box"
 Date "2020-10-12"

Commit message: Fixed Broken Library References
Connections:
- new net: A1.~ (~~D9), U9.~ (Serial_Clock) (x5)
Changed lines of the file:
@@
 EESchema Schematic File Version 4
+LIBS:Master System Schematic-cache
 EELAYER 30 0
 EELAYER END

Commit message: Clean up for merge
>cleaned wire runs on top sheet
Connections:
- new net: A1.~ (~~D9), U9.~ (Serial_Clock) (x5)
Changed lines of the file:
@@
 EESchema Schematic File Version 4
-LIBS:Master System Schematic-cache
 EELAYER 30 0
 EELAYER END
 $Descr A 11000 8500
 encoding utf-8
-Sheet 12 17
+Sheet 6 17
 Title "Pedal Box"
 Date "2020-10-12"
