File: Schematics/Master System Schematic/Brake Light.sch (KiCad schematic (older format))
At the start: 3 parts, among them U13 CAN_Bus_Module, U15 KY-019

Commit message: Driver IO Indicators and Toggle
Added Toggle Switch and LED indicators for BMS and IMD to master sheet and connections into Driver IO Box
Connections:
- new net: A3.~ (~~D9), U13.~ (Serial_Clock) (x6)
Changed lines of the file:
@@
 EESchema Schematic File Version 4
-LIBS:Master System Schematic-cache
 EELAYER 30 0
 EELAYER END

Commit message: Added cooling pump off while charging functionality
>Added diode so glv battery cannot supply charging power to bms
>added pulldown resistor for charging power line to ground
>Connected charging power line to second side of cooling pump relay coil
Connections:
- new net: A3.~ (~~D9), U13.~ (Serial_Clock) (x6)
Changed lines of the file:
@@
 $Descr A4 11693 8268
 encoding utf-8
-Sheet 21 21
+Sheet 20 21
 Title ""
 Date "2020-10-12"

Commit message: Fixed annotations and date
Connections:
- new net: A3.~ (~~D9), U13.~ (Serial_Clock) (x6)
Changed lines of the file:
@@
 EESchema Schematic File Version 4
+LIBS:Master System Schematic-cache
 EELAYER 30 0
 EELAYER END

Commit message: Fixed Issues from last update
Sent the toggle - to the 5v, made connections between BMS/IMD Fault (formerly just called indicator) pins and the BMD/IMD + pins
Connections:
- new net: A3.~ (~~D9), U13.~ (Serial_Clock) (x6)
Changed lines of the file:
@@
 EESchema Schematic File Version 4
-LIBS:Master System Schematic-cache
 EELAYER 30 0
 EELAYER END
